File: pcb/MiPi/MiPi.kicad_pcb (KiCad board)
At the start: 2 copper layers, 53 x 53 mm, 91 parts, among them J1 Micro_SD_Card, J2 AudioJack3, J3 USB_C_Receptacle_USB2.0_14P, Q1 Si1308EDL, SW1 SW_Push, SW2 SW_Push, SW3 RotaryEncoder_Switch_MP, SW4 SW_Push, SW5 SW_Push, SW6 SW_Push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

Commit message: Made the Gerbers, BOM, and CDL for the first version of miPi
Routing:
- net +3.3V: track 282.1 -> 282.9 mm
- net GND: vias 34 -> 66
Other:
- board text added: "12.2025 Rev.: 1"
